File: first_keeb/Electrical/first_keeb.kicad_sch (KiCad schematic)
At the start: 0 parts

Commit message: add MCU, i2c pullup, and oled to sch
Parts:
- added R0, R1: 10k, symbol Device:R
- added S1: SSD1306, symbol SSD1306-128x64_OLED:SSD1306
- added U1: Pico, RPi_Pico:RPi_Pico_SMD_TH, symbol MCU_RaspberryPi_and_Boards:Pico
- added U2: LM4040DBZ-3, Package_TO_SOT_SMD:SOT-23, symbol Reference_Voltage:LM4040DBZ-3
Connections:
- new net: U1.35 (ADC_VREF), U2.1 (K)
- new net +3V3: R0.1, R1.1, S1.2 (VCC), U1.36 (3V3)
- new net GND: S1.1 (GND), U2.2 (A)
- new net I2C0_SCL: R0.2, S1.3 (SCL), U1.24 (GPIO18)
- new net I2C0_SDA: R1.2, S1.4 (SDA), U1.25 (GPIO19)
Other:
- note added: "I2C Pullups"
- note added: "MCU breakout"
- note added: "OLED"
