File: first_keeb/Electrical/v4_proto/pcb/RP2040_minimal.kicad_pcb (KiCad board)
At the start: 2 copper layers, 80 x 80 mm, 68 parts, among them P1 USB4105-GF-A, Q1 SN74LV1T34DBV, SW1 SW_Push, SW2 SW_Push, SW3 SKRKAGE020, U1 NCP1117-3.3_SOT223, U2 LM4040DBZ-3, U3 PRTR5V0U2X, U4 W25Q32JVSS, U5 RP2040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

Commit message: creates a board that uses mid-mount usbc receptacle, and has all the rp2040 circuitry on the opposite layer of keyboard switches so that foam mod can be made easily. Also adds the threaded inserts
Parts:
- H3, H4, H6, H7: moved to F.Cu
- moved H4 56.0 mm to (72.0, 117.0), turned to 0 degrees
- moved H6 56.0 mm to (128.0, 117.0), turned to 0 degrees
- moved H3 35.0 mm to (82.5, 72.0), turned to 0 degrees
- moved H7 35.0 mm to (117.5, 72.0), turned to 0 degrees
Changed lines of the file:
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@@
     )
+  )
+  (footprint "MountingHole:M3_Threaded_Insert" (layer "F.Cu")
+    (at 128 117)
+    (property "Sheetfile" "RP2040_minimal.kicad_sch")
+    (property "Sheetname" "")
+    (property "ki_description" "Mounting Hole with connection")
+    (property "ki_keywords" "mounting hole")
+    (attr smd)
+    (fp_text reference "H6" (at 0 -0.5 unlocked) (layer "F.SilkS")
+        (effects (font (size 1 1) (thickness 0.15)))
+    )
+    (fp_text value "M3_Threaded_Insert" (at 0 1 unlocked) (layer "F.Fab")
+        (effects (font (size 1 1) (thickness 0.15)))
+    )
+    (fp_text user "${REFERENCE}" (at 0 2.5 unlocked) (layer "F.Fab")
+        (effects (font (size 1 1) (thickness 0.15)))
+    )
+    (fp_circle (center 0 0) (end 3.2 0)
+      (stroke (width 0.12) (type default)) (fill none) (layer "Cmts.User"))
+    (pad "" np_thru_hole circle (at 0 0) (size 4.2 4.2) (drill 4.2) (layers "F&B.Cu" "*.Mask"))
+    (pad "1" smd circle (at 0 0) (size 6.2 6.2) (layers "F.Cu" "F.Mask"))
   )
   (footprint "Capacitor_SMD:C_0402_1005Metric" (layer "F.Cu")
@@
     )
   )
+  (footprint "MountingHole:M3_Threaded_Insert" (layer "F.Cu")
+    (at 72 117)
+    (property "Sheetfile" "RP2040_minimal.kicad_sch")
+    (property "Sheetname" "")
+    (property "ki_description" "Mounting Hole with connection")
+    (property "ki_keywords" "mounting hole")
+    (attr smd)
+    (fp_text reference "H4" (at 0 -0.5 unlocked) (layer "F.SilkS")
+        (effects (font (size 1 1) (thickness 0.15)))
+    )
+    (fp_text value "M3_Threaded_Insert" (at 0 1 unlocked) (layer "F.Fab")
+        (effects (font (size 1 1) (thickness 0.15)))
+    )
+    (fp_text user "${REFERENCE}" (at 0 2.5 unlocked) (layer "F.Fab")
+        (effects (font (size 1 1) (thickness 0.15)))
+    )
+    (fp_circle (center 0 0) (end 3.2 0)
+      (stroke (width 0.12) (type default)) (fill none) (layer "Cmts.User"))
+    (pad "" np_thru_hole circle (at 0 0) (size 4.2 4.2) (drill 4.2) (layers "F&B.Cu" "*.Mask"))
+    (pad "1" smd circle (at 0 0) (size 6.2 6.2) (layers "F.Cu" "F.Mask"))
+  )
+  (footprint "MountingHole:M3_Threaded_Insert" (layer "F.Cu")
+    (at 82.5 72)
+    (property "Sheetfile" "RP2040_minimal.kicad_sch")
+    (property "Sheetname" "")
+    (property "ki_description" "Mounting Hole with connection")
+    (property "ki_keywords" "mounting hole")
+    (attr smd)
+    (fp_text reference "H3" (at 0 -0.5 unlocked) (layer "F.SilkS")
+        (effects (font (size 1 1) (thickness 0.15)))
+    )
+    (fp_text value "M3_Threaded_Insert" (at 0 1 unlocked) (layer "F.Fab")
+        (effects (font (size 1 1) (thickness 0.15)))
+    )
+    (fp_text user "${REFERENCE}" (at 0 2.5 unlocked) (layer "F.Fab")
+        (effects (font (size 1 1) (thickness 0.15)))
+    )
+    (fp_circle (center 0 0) (end 3.2 0)
+      (stroke (width 0.12) (type default)) (fill none) (layer "Cmts.User"))
+    (pad "" np_thru_hole circle (at 0 0) (size 4.2 4.2) (drill 4.2) (layers "F&B.Cu" "*.Mask"))
+    (pad "1" smd circle (at 0 0) (size 6.2 6.2) (layers "F.Cu" "F.Mask"))
+  )
   (footprint "LED_SMD:LED_WS2812B-2020_PLCC4_2.0x2.0mm" (layer "F.Cu")
     (at 77 75)
@@
     )
   )
+  (footprint "MountingHole:M3_Threaded_Insert" (layer "F.Cu")
+    (at 117.5 72)
+    (property "Sheetfile" "RP2040_minimal.kicad_sch")
+    (property "Sheetname" "")
+    (property "ki_description" "Mounting Hole with connection")
+    (property "ki_keywords" "mounting hole")
+    (attr smd)
+    (fp_text reference "H7" (at 0 -0.5 unlocked) (layer "F.SilkS")
+        (effects (font (size 1 1) (thickness 0.15)))
+    )
+    (fp_text value "M3_Threaded_Insert" (at 0 1 unlocked) (layer "F.Fab")
+        (effects (font (size 1 1) (thickness 0.15)))
+    )
+    (fp_text user "${REFERENCE}" (at 0 2.5 unlocked) (layer "F.Fab")
+        (effects (font (size 1 1) (thickness 0.15)))
+    )
+    (fp_circle (center 0 0) (end 3.2 0)
+      (stroke (width 0.12) (type default)) (fill none) (layer "Cmts.User"))
+    (pad "" np_thru_hole circle (at 0 0) (size 4.2 4.2) (drill 4.2) (layers "F&B.Cu" "*.Mask"))
+    (pad "1" smd circle (at 0 0) (size 6.2 6.2) (layers "F.Cu" "F.Mask"))
+  )
   (footprint "Package_TO_SOT_SMD:SOT-23-5" (layer "F.Cu")
     (at 69.7525 92.19 180)
@@
   )
   (footprint "MountingHole:M3_Threaded_Insert" (layer "B.Cu")
-    (at 72 117 180)
+    (at 128 83 180)
     (property "Sheetfile" "RP2040_minimal.kicad_sch")
     (property "Sheetname" "")
@@
     (property "ki_keywords" "mounting hole")
     (attr smd)
-    (fp_text reference "H6" (at 0 0.5 unlocked) (layer "B.SilkS")
-        (effects (font (size 1 1) (thickness 0.15)) (justify mirror))
-    )
-    (fp_text value "M3_Threaded_Insert" (at 0 -1 unlocked) (layer "B.Fab")
-        (effects (font (size 1 1) (thickness 0.15)) (justify mirror))
-    )
-    (fp_text user "${REFERENCE}" (at 0 -2.5 unlocked) (layer "B.Fab")
-        (effects (font (size 1 1) (thickness 0.15)) (justify mirror))
-    )
-    (fp_circle (center 0 0) (end 3.2 0)
-      (stroke (width 0.12) (type default)) (fill none) (layer "Cmts.User"))
-    (pad "" np_thru_hole circle (at 0 0 180) (size 4.2 4.2) (drill 4.2) (layers "F&B.Cu" "*.Mask"))
-    (pad "1" smd circle (at 0 0 180) (size 6.2 6.2) (layers "B.Cu" "B.Mask"))
-  )
-  (footprint "MountingHole:M3_Threaded_Insert" (layer "B.Cu")
-    (at 128 83 180)
-    (property "Sheetfile" "RP2040_minimal.kicad_sch")
-    (property "Sheetname" "")
-    (property "ki_description" "Mounting Hole with connection")
-    (property "ki_keywords" "mounting hole")
-    (attr smd)
     (fp_text reference "H1" (at 0 0.5 unlocked) (layer "B.SilkS")
-        (effects (font (size 1 1) (thickness 0.15)) (justify mirror))
-    )
-    (fp_text value "M3_Threaded_Insert" (at 0 -1 unlocked) (layer "B.Fab")
-        (effects (font (size 1 1) (thickness 0.15)) (justify mirror))
-    )
-    (fp_text user "${REFERENCE}" (at 0 -2.5 unlocked) (layer "B.Fab")
-        (effects (font (size 1 1) (thickness 0.15)) (justify mirror))
-    )
-    (fp_circle (center 0 0) (end 3.2 0)
-      (stroke (width 0.12) (type default)) (fill none) (layer "Cmts.User"))
-    (pad "" np_thru_hole circle (at 0 0 180) (size 4.2 4.2) (drill 4.2) (layers "F&B.Cu" "*.Mask"))
-    (pad "1" smd circle (at 0 0 180) (size 6.2 6.2) (layers "B.Cu" "B.Mask"))
-  )
-  (footprint "MountingHole:M3_Threaded_Insert" (layer "B.Cu")
-    (at 128 117 180)
-    (property "Sheetfile" "RP2040_minimal.kicad_sch")
-    (property "Sheetname" "")
-    (property "ki_description" "Mounting Hole with connection")
-    (property "ki_keywords" "mounting hole")
-    (attr smd)
-    (fp_text reference "H4" (at 0 0.5 unlocked) (layer "B.SilkS")
         (effects (font (size 1 1) (thickness 0.15)) (justify mirror))
     )
@@
     )
   )
-  (footprint "MountingHole:M3_Threaded_Insert" (layer "B.Cu")
-    (at 117.5 72 180)
-    (property "Sheetfile" "RP2040_minimal.kicad_sch")
-    (property "Sheetname" "")
-    (property "ki_description" "Mounting Hole with connection")
-    (property "ki_keywords" "mounting hole")
-    (attr smd)
-    (fp_text reference "H3" (at 0 0.5 unlocked) (layer "B.SilkS")
-        (effects (font (size 1 1) (thickness 0.15)) (justify mirror))
-    )
-    (fp_text value "M3_Threaded_Insert" (at 0 -1 unlocked) (layer "B.Fab")
-        (effects (font (size 1 1) (thickness 0.15)) (justify mirror))
-    )
-    (fp_text user "${REFERENCE}" (at 0 -2.5 unlocked) (layer "B.Fab")
-        (effects (font (size 1 1) (thickness 0.15)) (justify mirror))
-    )
-    (fp_circle (center 0 0) (end 3.2 0)
-      (stroke (width 0.12) (type default)) (fill none) (layer "Cmts.User"))
-    (pad "" np_thru_hole circle (at 0 0 180) (size 4.2 4.2) (drill 4.2) (layers "F&B.Cu" "*.Mask"))
-    (pad "1" smd circle (at 0 0 180) (size 6.2 6.2) (layers "B.Cu" "B.Mask"))
-  )
-  (footprint "MountingHole:M3_Threaded_Insert" (layer "B.Cu")
-    (at 82.5 72 180)
-    (property "Sheetfile" "RP2040_minimal.kicad_sch")
-    (property "Sheetname" "")
-    (property "ki_description" "Mounting Hole with connection")
-    (property "ki_keywords" "mounting hole")
-    (attr smd)
-    (fp_text reference "H7" (at 0 0.5 unlocked) (layer "B.SilkS")
-        (effects (font (size 1 1) (thickness 0.15)) (justify mirror))
-    )
-    (fp_text value "M3_Threaded_Insert" (at 0 -1 unlocked) (layer "B.Fab")
-        (effects (font (size 1 1) (thickness 0.15)) (justify mirror))
-    )
-    (fp_text user "${REFERENCE}" (at 0 -2.5 unlocked) (layer "B.Fab")
-        (effects (font (size 1 1) (thickness 0.15)) (justify mirror))
-    )
-    (fp_circle (center 0 0) (end 3.2 0)
-      (stroke (width 0.12) (type default)) (fill none) (layer "Cmts.User"))
-    (pad "" np_thru_hole circle (at 0 0 180) (size 4.2 4.2) (drill 4.2) (layers "F&B.Cu" "*.Mask"))
-    (pad "1" smd circle (at 0 0 180) (size 6.2 6.2) (layers "B.Cu" "B.Mask"))
-  )
   (gr_circle (center 100 100) (end 136 100)
