File: first_keeb/Electrical/v7_proto_standoff_and_nuts/2_layer_pcb/RP2040_minimal.kicad_sch (KiCad schematic)
At the start: 63 parts, among them P1 USB-TYPE-C-016, Q1 SN74LV1T34DBV, SW1 SKRKAGE020, SW2 PTS647 SN70 SMTR2 LFS, SW3 PTS647 SN70 SMTR2 LFS, U1 NCP1117-3.3_SOT223, U2 LM4040DBZ-3, U3 PRTR5V0U2X, U4 W25Q32JVSS, U5 RP2040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

Commit message: adds 2 layer and 4 layer pcb versions
Parts:
- added R9: 1k, Capacitor_SMD:C_0402_1005Metric, symbol Device:R
- SW1: value SKRKAGE020 -> SKRKAHE020
Connections:
- net QSPI_SS: now also R9.2; no longer SW1.2
- new net: R9.1, SW1.2
Other:
- note removed: "Power"
- company: Raspberry Pi (Trading) Ltd -> (none)
- title: RP2040 Minimal Design Example -> keeb
- moved on the sheet: SW1
Changed lines of the file:
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@@
   (paper "A3")
   (title_block
-    (title "RP2040 Minimal Design Example")
+    (title "keeb")
     (date "2020-12-18")
     (rev "REV1")
-    (company "Raspberry Pi (Trading) Ltd")
   )
   (junction (at 172.085 65.405) (diameter 0) (color 0 0 0 0)
@@
   (junction (at 186.055 65.405) (diameter 0) (color 0 0 0 0)
   )
-  (junction (at 259.08 112.395) (diameter 0) (color 0 0 0 0)
-  )
   (junction (at 267.97 216.535) (diameter 0) (color 0 0 0 0)
   )
@@
   (junction (at 250.19 55.245) (diameter 0) (color 0 0 0 0)
   )
+  (junction (at 259.08 112.395) (diameter 0) (color 0 0 0 0)
+  )
   (junction (at 128.27 36.83) (diameter 0) (color 0 0 0 0)
   )
@@
     (stroke (width 0) (type default))
   )
-  (wire (pts (xy 240.03 112.395) (xy 240.03 115.57))
+  (wire (pts (xy 225.425 112.395) (xy 225.425 115.57))
     (stroke (width 0) (type default))
   )
@@
     (stroke (width 0) (type default))
   )
-  (wire (pts (xy 250.19 112.395) (xy 259.08 112.395))
-    (stroke (width 0) (type default))
-  )
   (wire (pts (xy 111.76 133.35) (xy 127 133.35))
     (stroke (width 0) (type default))
@@
     (stroke (width 0) (type default))
   )
+  (wire (pts (xy 252.095 112.395) (xy 259.08 112.395))
+    (stroke (width 0) (type default))
+  )
   (wire (pts (xy 111.76 156.21) (xy 128.905 156.21))
     (stroke (width 0) (type default))
@@
     (stroke (width 0) (type default))
   )
+  (wire (pts (xy 235.585 112.395) (xy 244.475 112.395))
+    (stroke (width 0) (type default))
+  )
   (wire (pts (xy 116.84 38.1) (xy 116.84 36.83))
     (stroke (width 0) (type default))
@@
     (effects (font (size 1 1)) (justify left bottom))
   )
-  (text "BOOTSEL" (at 240.03 102.87 0)
+  (text "BOOTSEL" (at 225.425 102.87 0)
     (effects (font (size 1.27 1.27)) (justify left bottom))
   )
-  (text "Power" (at 240.03 16.51 0)
-    (effects (font (size 2.54 2.54)) (justify left bottom))
-  )
   (text "Buttons" (at 66.04 245.11 0)
     (effects (font (size 2 2)) (justify left bottom))
@@
     )
   )
+  (symbol (lib_id "Device:R") (at 248.285 112.395 90) (unit 1)
+    (in_bom yes) (on_board yes) (dnp no) (fields_autoplaced)
+    (property "Reference" "R9" (at 248.285 107.95 90)
+      (effects (font (size 1.27 1.27)))
+    )
+    (property "Value" "1k" (at 248.285 110.49 90)
+      (effects (font (size 1.27 1.27)))
+    )
+    (property "Footprint" "Capacitor_SMD:C_0402_1005Metric" (at 248.285 114.173 90)
+      (effects (font (size 1.27 1.27)) hide)
+    )
+    (property "Datasheet" "~" (at 248.285 112.395 0)
+      (effects (font (size 1.27 1.27)) hide)
+    )
+    (pin "1")
+    (pin "2")
+    (instances
+      (project "RP2040_minimal"
+        (path "/26e500cb-9f3f-4e62-bb26-21a6be4a5bcc"
+          (reference "R9") (unit 1)
+        )
+      )
+    )
+  )
   (symbol (lib_id "power:+5V") (at 239.395 214.63 0) (unit 1)
     (in_bom yes) (on_board yes) (dnp no)
@@
     )
   )
-  (symbol (lib_id "power:GND") (at 240.03 115.57 0) (unit 1)
+  (symbol (lib_id "power:GND") (at 225.425 115.57 0) (unit 1)
     (in_bom yes) (on_board yes) (dnp no)
-    (property "Reference" "#PWR022" (at 240.03 121.92 0)
+    (property "Reference" "#PWR022" (at 225.425 121.92 0)
       (effects (font (size 1.27 1.27)) hide)
     )
-    (property "Value" "GND" (at 243.84 116.84 0)
+    (property "Value" "GND" (at 229.235 116.84 0)
       (effects (font (size 1.27 1.27)))
     )
-    (property "Footprint" "" (at 240.03 115.57 0)
+    (property "Footprint" "" (at 225.425 115.57 0)
       (effects (font (size 1.27 1.27)) hide)
     )
-    (property "Datasheet" "" (at 240.03 115.57 0)
+    (property "Datasheet" "" (at 225.425 115.57 0)
       (effects (font (size 1.27 1.27)) hide)
     )
@@
     )
   )
-  (symbol (lib_id "Switch:SW_Push") (at 245.11 112.395 0) (unit 1)
+  (symbol (lib_id "Switch:SW_Push") (at 230.505 112.395 0) (unit 1)
     (in_bom yes) (on_board yes) (dnp no) (fields_autoplaced)
-    (property "Reference" "SW1" (at 245.11 105.41 0)
+    (property "Reference" "SW1" (at 230.505 105.41 0)
       (effects (font (size 1.27 1.27)))
     )
-    (property "Value" "SKRKAGE020" (at 245.11 107.95 0)
+    (property "Value" "SKRKAHE020" (at 230.505 107.95 0)
       (effects (font (size 1.27 1.27)))
     )
-    (property "Footprint" "Button_Switch_SMD:SW_Push_SPST_NO_Alps_SKRK" (at 245.11 107.315 0)
+    (property "Footprint" "Button_Switch_SMD:SW_Push_SPST_NO_Alps_SKRK" (at 230.505 107.315 0)
       (effects (font (size 1.27 1.27)) hide)
     )
-    (property "Datasheet" "~" (at 245.11 107.315 0)
+    (property "Datasheet" "~" (at 230.505 107.315 0)
       (effects (font (size 1.27 1.27)) hide)
     )
