File: first_keeb/Electrical/v1_proto_standoff_and_nuts/pcb/RP2040_minimal.kicad_pcb (KiCad board)
At the start: 4 copper layers, 67.1 x 66.8 mm, 81 parts, among them J1 Conn_01x04_Socket, P1 USB-TYPE-C-016, Q1 SN74LV1T34DBV, SW1 SK-3296S-01-L3, SW2 MS-22C01-G010, SW3 TS-1187A-B-A-B, SW4 MS-22C01-G010, SW5 TS-1187A-B-A-B, SW6 BUTT1, SW7 BUTT3, SW8 BUTT2, U1 ME6206A25XG, U2 ME6208A44M3G, U3 PRTR5V0U2X, U4 MCP6001-OT, U5 STM32F401RCTx, U6 MCP6001-OT, U7 SLSS49E, U8 SLSS49E, U9 SLSS49E, Y1 8MHz

Commit message: fix mag sensor schematic
Routing:
- net GND: track 120.7 -> 120.6 mm, vias 337 -> 346
Changed lines of the file:
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@@
       (net 84 "+4V4") (pinfunction "VCC") (pintype "power_in"))
     (pad "2" smd roundrect (at -0.9375 0.95 180) (size 1.475 0.6) (layers "F.Cu" "F.Paste" "F.Mask") (roundrect_rratio 0.25)
-      (net 89 "S_ADC_IN3") (pinfunction "GND") (pintype "open_collector"))
+      (net 89 "S_ADC_IN3") (pinfunction "VOUT") (pintype "open_collector"))
     (pad "3" smd roundrect (at 0.9375 0 180) (size 1.475 0.6) (layers "F.Cu" "F.Paste" "F.Mask") (roundrect_rratio 0.25)
-      (net 1 "GND") (pinfunction "Vout") (pintype "power_in"))
+      (net 1 "GND") (pinfunction "GND") (pintype "power_in"))
     (model "${KICAD6_3DMODEL_DIR}/Package_TO_SOT_SMD.3dshapes/SOT-23.wrl"
       (offset (xyz 0 0 0))
@@
       (net 84 "+4V4") (pinfunction "VCC") (pintype "power_in"))
     (pad "2" smd roundrect (at -0.9375 0.95 270) (size 1.475 0.6) (layers "F.Cu" "F.Paste" "F.Mask") (roundrect_rratio 0.25)
-      (net 86 "S_ADC_IN2") (pinfunction "GND") (pintype "open_collector"))
+      (net 86 "S_ADC_IN2") (pinfunction "VOUT") (pintype "open_collector"))
     (pad "3" smd roundrect (at 0.9375 0 270) (size 1.475 0.6) (layers "F.Cu" "F.Paste" "F.Mask") (roundrect_rratio 0.25)
-      (net 1 "GND") (pinfunction "Vout") (pintype "power_in"))
+      (net 1 "GND") (pinfunction "GND") (pintype "power_in"))
     (model "${KICAD6_3DMODEL_DIR}/Package_TO_SOT_SMD.3dshapes/SOT-23.wrl"
       (offset (xyz 0 0 0))
@@
       (net 84 "+4V4") (pinfunction "VCC") (pintype "power_in"))
     (pad "2" smd roundrect (at -0.9375 0.95 180) (size 1.475 0.6) (layers "F.Cu" "F.Paste" "F.Mask") (roundrect_rratio 0.25)
-      (net 18 "ADC_IN1") (pinfunction "GND") (pintype "open_collector"))
+      (net 18 "ADC_IN1") (pinfunction "VOUT") (pintype "open_collector"))
     (pad "3" smd roundrect (at 0.9375 0 180) (size 1.475 0.6) (layers "F.Cu" "F.Paste" "F.Mask") (roundrect_rratio 0.25)
-      (net 1 "GND") (pinfunction "Vout") (pintype "power_in"))
+      (net 1 "GND") (pinfunction "GND") (pintype "power_in"))
     (model "${KICAD6_3DMODEL_DIR}/Package_TO_SOT_SMD.3dshapes/SOT-23.wrl"
       (offset (xyz 0 0 0))
@@
   (segment (start 81.625 92.825) (end 82.47 92.825) (width 0.3) (layer "F.Cu") (net 1))
   (segment (start 111.172973 79.1) (end 111.025 79.1) (width 0.6) (layer "F.Cu") (net 1))
-  (segment (start 100 100.9375) (end 100 102.08) (width 0.3) (layer "F.Cu") (net 1))
   (segment (start 79.39 84.995) (end 79.39 86.395) (width 0.3) (layer "F.Cu") (net 1))
   (segment (start 78.945 86.755) (end 79.75 86.755) (width 0.3) (layer "F.Cu") (net 1))
@@
   (segment (start 95.479259 73.467682) (end 95.764073 73.467682) (width 0.3) (layer "F.Cu") (net 1))
   (segment (start 88.355 78.3) (end 88.285 78.37) (width 0.3) (layer "F.Cu") (net 1))
-  (segment (start 100 102.08) (end 99.74 102.34) (width 0.3) (layer "F.Cu") (net 1))
   (segment (start 105.18 113.94) (end 105.1325 113.93) (width 0.6) (layer "F.Cu") (net 1))
   (segment (start 97.742086 90.57) (end 98.64 90.57) (width 0.3) (layer "F.Cu") (net 1))
   (segment (start 94.65 92.201041) (end 94.898959 92.45) (width 0.3) (layer "F.Cu") (net 1))
   (segment (start 87.9 77.425) (end 88.355 77.88) (width 0.3) (layer "F.Cu") (net 1))
-  (segment (start 99.74 102.38) (end 99.7 102.38) (width 0.3) (layer "F.Cu") (net 1))
   (segment (start 86.69 93.21) (end 86.71 93.21) (width 0.3) (layer "F.Cu") (net 1))
   (segment (start 122.31 102.2) (end 121.34 102.2) (width 0.3) (layer "F.Cu") (net 1))
   (segment (start 105.38 84.58) (end 105.38 84.62) (width 0.3) (layer "F.Cu") (net 1))
   (segment (start 83.34 82.21) (end 83.23 82.1) (width 0.3) (layer "F.Cu") (net 1))
-  (segment (start 99.74 102.34) (end 99.74 102.38) (width 0.3) (layer "F.Cu") (net 1))
   (segment (start 109.205 81.675) (end 109.205 82.805) (width 0.6) (layer "F.Cu") (net 1))
   (segment (start 103.8 73.95) (end 103.72 73.87) (width 0.3) (layer "F.Cu") (net 1))
   (segment (start 112.69 94.02) (end 112.85 94.02) (width 0.3) (layer "F.Cu") (net 1))
   (segment (start 95.66 94.958959) (end 95.61 95.008959) (width 0.3) (layer "F.Cu") (net 1))
-  (segment (start 99.7 102.38) (end 99.83 102.25) (width 0.3) (layer "F.Cu") (net 1))
   (segment (start 110.293813 83.302187) (end 109.225 83.302187) (width 0.6) (layer "F.Cu") (net 1))
   (segment (start 106.855 113.94) (end 105.18 113.94) (width 0.6) (layer "F.Cu") (net 1))
@@
   (segment (start 112.265 79.1) (end 112.275 79.09) (width 0.6) (layer "F.Cu") (net 1))
   (segment (start 95.59 95.028959) (end 95.66 95.028959) (width 0.3) (layer "F.Cu") (net 1))
+  (segment (start 99.7 102.38) (end 99.83 102.25) (width 0.3) (layer "F.Cu") (net 1))
   (segment (start 83.18 102.78) (end 83.02 102.78) (width 0.3) (layer "F.Cu") (net 1))
   (segment (start 98.2 81.648959) (end 98.2 82.151041) (width 0.3) (layer "F.Cu") (net 1))
@@
   (segment (start 95.88 74.14) (end 95.88 74.2) (width 0.6) (layer "F.Cu") (net 1))
   (segment (start 82.32 85.65) (end 82.44 85.53) (width 0.3) (layer "F.Cu") (net 1))
+  (segment (start 100 102.08) (end 100 100.9375) (width 0.3) (layer "F.Cu") (net 1))
   (segment (start 108.545 113.93) (end 108.555 113.93) (width 0.6) (layer "F.Cu") (net 1))
   (segment (start 116.81 100.02) (end 116.81 100.06) (width 0.3) (layer "F.Cu") (net 1))
@@
   (segment (start 96.028959 92.45) (end 96.11 92.368959) (width 0.3) (layer "F.Cu") (net 1))
   (segment (start 83.21 85.51) (end 82.46 85.51) (width 0.3) (layer "F.Cu") (net 1))
+  (segment (start 99.7 102.38) (end 100 102.08) (width 0.3) (layer "F.Cu") (net 1))
   (segment (start 95.88 74.2) (end 95.82 74.2) (width 0.6) (layer "F.Cu") (net 1))
   (via (at 108.21 102.33) (size 0.8) (drill 0.4) (layers "F.Cu" "B.Cu") (free) (net 1))
@@
   (via (at 81.9 81.175) (size 0.8) (drill 0.4) (layers "F.Cu" "B.Cu") (net 1))
   (via (at 78.24 87.7) (size 0.8) (drill 0.4) (layers "F.Cu" "B.Cu") (net 1))
+  (via (at 122.7 97.725) (size 0.8) (drill 0.4) (layers "F.Cu" "B.Cu") (free) (net 1))
   (via (at 82.16 75.76) (size 0.8) (drill 0.4) (layers "F.Cu" "B.Cu") (net 1))
   (via (at 97.79 117.094) (size 0.8) (drill 0.4) (layers "F.Cu" "B.Cu") (net 1))
@@
   (via (at 95.479259 73.467682) (size 0.8) (drill 0.4) (layers "F.Cu" "B.Cu") (net 1))
   (via (at 110.998 89.916) (size 0.8) (drill 0.4) (layers "F.Cu" "B.Cu") (free) (net 1))
+  (via (at 122.675 100.775) (size 0.8) (drill 0.4) (layers "F.Cu" "B.Cu") (free) (net 1))
   (via (at 114.52 102.47) (size 0.8) (drill 0.4) (layers "F.Cu" "B.Cu") (free) (net 1))
   (via (at 103.124 88.9) (size 0.8) (drill 0.4) (layers "F.Cu" "B.Cu") (free) (net 1))
   (via (at 104.75 97.925) (size 0.8) (drill 0.4) (layers "F.Cu" "B.Cu") (free) (net 1))
   (via (at 86.25 112.2) (size 0.8) (drill 0.4) (layers "F.Cu" "B.Cu") (free) (net 1))
-  (via (at 99.74 102.38) (size 0.8) (drill 0.4) (layers "F.Cu" "B.Cu") (net 1))
+  (via (at 99.7 102.38) (size 0.8) (drill 0.4) (layers "F.Cu" "B.Cu") (net 1))
   (via (at 93.472 106.426) (size 0.8) (drill 0.4) (layers "F.Cu" "B.Cu") (free) (net 1))
   (via (at 105.38 84.58) (size 0.8) (drill 0.4) (layers "F.Cu" "B.Cu") (net 1))
@@
   (via (at 114.49 90.63) (size 0.8) (drill 0.4) (layers "F.Cu" "B.Cu") (free) (net 1))
   (via (at 124.05 103.625) (size 0.8) (drill 0.4) (layers "F.Cu" "B.Cu") (free) (net 1))
+  (via (at 121.375 97.45) (size 0.8) (drill 0.4) (layers "F.Cu" "B.Cu") (free) (net 1))
   (via (at 105.58 104.54) (size 0.8) (drill 0.4) (layers "F.Cu" "B.Cu") (free) (net 1))
   (via (at 95.5 86.375) (size 0.8) (drill 0.4) (layers "F.Cu" "B.Cu") (free) (net 1))
   (via (at 81.31 102.64) (size 0.8) (drill 0.4) (layers "F.Cu" "B.Cu") (free) (net 1))
   (via (at 101.985023 75.724977) (size 0.8) (drill 0.4) (layers "F.Cu" "B.Cu") (net 1))
+  (via (at 122.825 99.4) (size 0.8) (drill 0.4) (layers "F.Cu" "B.Cu") (free) (net 1))
   (via (at 95.68 88.36) (size 0.8) (drill 0.4) (layers "F.Cu" "B.Cu") (free) (net 1))
+  (via (at 107.05 101.025) (size 0.8) (drill 0.4) (layers "F.Cu" "B.Cu") (free) (net 1))
   (via (at 97.26 75.86) (size 0.8) (drill 0.4) (layers "F.Cu" "B.Cu") (net 1))
   (via (at 87.3 95.12) (size 0.8) (drill 0.4) (layers "F.Cu" "B.Cu") (free) (net 1))
@@
   (via (at 113.56 92.34) (size 0.8) (drill 0.4) (layers "F.Cu" "B.Cu") (free) (net 1))
   (via (at 118.5 77.075) (size 0.8) (drill 0.4) (layers "F.Cu" "B.Cu") (free) (net 1))
+  (via (at 78.475 97.05) (size 0.8) (drill 0.4) (layers "F.Cu" "B.Cu") (free) (net 1))
   (via (at 109.23 88.67) (size 0.8) (drill 0.4) (layers "F.Cu" "B.Cu") (free) (net 1))
   (via (at 102.87 87.63) (size 0.8) (drill 0.4) (layers "F.Cu" "B.Cu") (free) (net 1))
@@
   (via (at 78.13 86.25) (size 0.8) (drill 0.4) (layers "F.Cu" "B.Cu") (net 1))
   (via (at 102.825 81.45) (size 0.8) (drill 0.4) (layers "F.Cu" "B.Cu") (free) (net 1))
+  (via (at 103.05 98.725) (size 0.8) (drill 0.4) (layers "F.Cu" "B.Cu") (free) (net 1))
   (via (at 91.45 83.5) (size 0.8) (drill 0.4) (layers "F.Cu" "B.Cu") (free) (net 1))
   (via (at 109.93 77.425) (size 0.8) (drill 0.4) (layers "F.Cu" "B.Cu") (net 1))
@@
   (via (at 89.56 112.69) (size 0.8) (drill 0.4) (layers "F.Cu" "B.Cu") (free) (net 1))
   (via (at 75.125 103.65) (size 0.8) (drill 0.4) (layers "F.Cu" "B.Cu") (free) (net 1))
+  (via (at 80.55 97.075) (size 0.8) (drill 0.4) (layers "F.Cu" "B.Cu") (free) (net 1))
   (via (at 87.35 86.625) (size 0.8) (drill 0.4) (layers "F.Cu" "B.Cu") (free) (net 1))
   (via (at 78.994 79.859502) (size 0.8) (drill 0.4) (layers "F.Cu" "B.Cu") (net 1))
   (via (at 74.168 84.074) (size 0.8) (drill 0.4) (layers "F.Cu" "B.Cu") (free) (net 1))
+  (via (at 82.15 96.975) (size 0.8) (drill 0.4) (layers "F.Cu" "B.Cu") (free) (net 1))
   (via (at 93.03 93.09) (size 0.8) (drill 0.4) (layers "F.Cu" "B.Cu") (free) (net 1))
   (segment (start 82.21 105.4) (end 82.2 105.4) (width 0.3) (layer "B.Cu") (net 1))

Commit message: add svg
Routing:
- net GND: vias 346 -> 353
Changed lines of the file:
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@@
   (via (at 103.812 118.11) (size 0.8) (drill 0.4) (layers "F.Cu" "B.Cu") (net 1))
   (via (at 117.09 102.51) (size 0.8) (drill 0.4) (layers "F.Cu" "B.Cu") (free) (net 1))
+  (via (at 73.95 90.95) (size 0.8) (drill 0.4) (layers "F.Cu" "B.Cu") (free) (net 1))
   (via (at 89.34 93.29) (size 0.8) (drill 0.4) (layers "F.Cu" "B.Cu") (free) (net 1))
   (via (at 100.584 87.884) (size 0.8) (drill 0.4) (layers "F.Cu" "B.Cu") (free) (net 1))
@@
   (via (at 84.836 110.744) (size 0.8) (drill 0.4) (layers "F.Cu" "B.Cu") (free) (net 1))
   (via (at 84.07 108.24) (size 0.8) (drill 0.4) (layers "F.Cu" "B.Cu") (free) (net 1))
+  (via (at 76.075 83.775) (size 0.8) (drill 0.4) (layers "F.Cu" "B.Cu") (free) (net 1))
   (via (at 110.293813 83.302187) (size 0.8) (drill 0.4) (layers "F.Cu" "B.Cu") (net 1))
   (via (at 107.08 104.58) (size 0.8) (drill 0.4) (layers "F.Cu" "B.Cu") (free) (net 1))
@@
   (via (at 99.96 92.51) (size 0.8) (drill 0.4) (layers "F.Cu" "B.Cu") (free) (net 1))
   (via (at 77.775 101.2) (size 0.8) (drill 0.4) (layers "F.Cu" "B.Cu") (free) (net 1))
+  (via (at 71.95 89.025) (size 0.8) (drill 0.4) (layers "F.Cu" "B.Cu") (free) (net 1))
   (via (at 104.425 79.975) (size 0.8) (drill 0.4) (layers "F.Cu" "B.Cu") (free) (net 1))
   (via (at 103.91 96.15) (size 0.8) (drill 0.4) (layers "F.Cu" "B.Cu") (free) (net 1))
@@
   (via (at 74.676 83.058) (size 0.8) (drill 0.4) (layers "F.Cu" "B.Cu") (free) (net 1))
   (via (at 104.76 102.39) (size 0.8) (drill 0.4) (layers "F.Cu" "B.Cu") (free) (net 1))
+  (via (at 72.925 89.15) (size 0.8) (drill 0.4) (layers "F.Cu" "B.Cu") (free) (net 1))
   (via (at 112.522 91.44) (size 0.8) (drill 0.4) (layers "F.Cu" "B.Cu") (free) (net 1))
   (via (at 77.775 98.5) (size 0.8) (drill 0.4) (layers "F.Cu" "B.Cu") (free) (net 1))
@@
   (via (at 75.893019 92.9805) (size 0.8) (drill 0.4) (layers "F.Cu" "B.Cu") (free) (net 1))
   (via (at 84.4 102.725) (size 0.8) (drill 0.4) (layers "F.Cu" "B.Cu") (free) (net 1))
+  (via (at 76.875 82.5) (size 0.8) (drill 0.4) (layers "F.Cu" "B.Cu") (free) (net 1))
   (via (at 106.15 73.5) (size 0.8) (drill 0.4) (layers "F.Cu" "B.Cu") (free) (net 1))
   (via (at 90.45 76.325) (size 0.8) (drill 0.4) (layers "F.Cu" "B.Cu") (free) (net 1))
@@
   (via (at 96.27 127.24) (size 0.8) (drill 0.4) (layers "F.Cu" "B.Cu") (net 1))
   (via (at 123.48 96.33) (size 0.8) (drill 0.4) (layers "F.Cu" "B.Cu") (free) (net 1))
+  (via (at 72.675 90.95) (size 0.8) (drill 0.4) (layers "F.Cu" "B.Cu") (free) (net 1))
   (via (at 87.02 97.56) (size 0.8) (drill 0.4) (layers "F.Cu" "B.Cu") (free) (net 1))
+  (via (at 75.7 90.925) (size 0.8) (drill 0.4) (layers "F.Cu" "B.Cu") (free) (net 1))
   (via (at 109.25 80.025) (size 0.8) (drill 0.4) (layers "F.Cu" "B.Cu") (free) (net 1))
   (via (at 93.68 112.8) (size 0.8) (drill 0.4) (layers "F.Cu" "B.Cu") (free) (net 1))
@@
   (segment (start 106.310001 127.364999) (end 105.660001 127.364999) (width 0.3) (layer "B.Cu") (net 4))
   (segment (start 100.587 117.052) (end 100.737 117.052) (width 0.3) (layer "B.Cu") (net 4))
+  (segment (start 72.052207 90.3) (end 72.372207 89.98) (width 0.6) (layer "F.Cu") (net 5))
   (segment (start 95.06 129.33) (end 88.944 129.33) (width 0.6) (layer "F.Cu") (net 5))
   (segment (start 100.010353 83.780354) (end 101.344646 83.780354) (width 0.4) (layer "F.Cu") (net 5))
@@
   (segment (start 112.325 75.22) (end 111.54 75.22) (width 0.6) (layer "F.Cu") (net 5))
   (segment (start 72.39 82.55) (end 78.63 76.31) (width 0.6) (layer "F.Cu") (net 5))
+  (segment (start 71.2 90.3) (end 72.052207 90.3) (width 0.6) (layer "F.Cu") (net 5))
   (segment (start 126.04 109.64) (end 123.5 112.18) (width 0.6) (layer "F.Cu") (net 5))
   (segment (start 102.108 115.316) (end 94.744793 115.316) (width 0.6) (layer "F.Cu") (net 5))
@@
   (segment (start 95.56 128.83) (end 94.9 128.17) (width 0.6) (layer "F.Cu") (net 5))
   (segment (start 125.89 109.79) (end 125.89 115.8) (width 0.6) (layer "F.Cu") (net 5))
-  (segment (start 70.37 91.13) (end 71.52 89.98) (width 0.6) (layer "F.Cu") (net 5))
   (segment (start 109.024793 130.048) (end 96.778 130.048) (width 0.6) (layer "F.Cu") (net 5))
   (segment (start 101.344646 83.780354) (end 101.44 83.685) (width 0.4) (layer "F.Cu") (net 5))
+  (segment (start 72.372207 89.98) (end 76.94 89.98) (width 0.6) (layer "F.Cu") (net 5))
   (segment (start 106.8725 110.925) (end 104.595 110.925) (width 0.6) (layer "F.Cu") (net 5))
   (segment (start 101.953629 82.935) (end 103.38 82.935) (width 0.4) (layer "F.Cu") (net 5))
+  (segment (start 70.37 91.13) (end 71.2 90.3) (width 0.6) (layer "F.Cu") (net 5))
   (segment (start 117.6 74.7) (end 121.14 78.24) (width 0.6) (layer "F.Cu") (net 5))
   (segment (start 93.614 115.174) (end 87.716793 115.174) (width 0.6) (layer "F.Cu") (net 5))
@@
   (segment (start 103.467207 113.956793) (end 102.108 115.316) (width 0.6) (layer "F.Cu") (net 5))
   (segment (start 126.04 109.64) (end 125.89 109.79) (width 0.6) (layer "F.Cu") (net 5))
-  (segment (start 71.52 89.98) (end 76.94 89.98) (width 0.6) (layer "F.Cu") (net 5))
   (segment (start 76.56 109.54) (end 76.56 115.19) (width 0.6) (layer "F.Cu") (net 5))
   (segment (start 95.56 128.83) (end 95.06 129.33) (width 0.6) (layer "F.Cu") (net 5))
